File: shoes.kicad_pcb (KiCad board)
At the start: 2 copper layers, 101 parts, among them P1 USB_OTG

Commit message: bakar and wires and shit
Parts:
- moved D51 174.0 mm to (95.2, 45.7)
- moved D88 171.3 mm to (118.1, 99.1)
- moved D69 169.8 mm to (102.9, 106.7)
- moved D48 163.4 mm to (87.6, 99.1)
- moved D52 160.7 mm to (95.2, 53.3)
- moved D97 159.4 mm to (125.7, 91.4)
- moved D83 157.6 mm to (118.1, 61.0)
- moved D100 156.4 mm to (125.7, 114.3)
- moved D39 155.0 mm to (80.0, 106.7)
- moved D58 153.2 mm to (95.2, 99.1)
- moved D46 153.1 mm to (87.6, 83.8)
- moved D82 150.7 mm to (118.1, 53.3)
- moved D92 149.6 mm to (125.7, 53.3)
- moved D99 148.0 mm to (125.7, 106.7)
- moved D37 147.4 mm to (80.0, 91.4)
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Routing:
- net Net-(D1-Pad2): track 0.00 -> 685.8 mm
- net VCC: track 0.00 -> 342.9 mm
- net GND: track 76.2 -> 350.5 mm

Commit message: WIP: added tracks
Parts:
- moved P1 108.1 mm to (92.7, 124.5)
Routing:
- net Net-(D1-Pad2): track 685.8 -> 839.0 mm
- net VCC: track 342.9 -> 401.1 mm, vias 0 -> 1
- net GND: track 350.5 -> 407.7 mm, vias 0 -> 1
Other:
- net class Default: clearance 0.2 -> 0.1
- rule trace_clearance: 0.2 -> 0.1
